Commit message: fixed odom, added ekf (needs tuning)

File: src/bb8_description/urdf/head.xacro (robot description, xacro)
@@ -11,10 +11,10 @@
       </material>
     </visual>
-    <!-- <collision>
+    <collision>
       <origin xyz="0 0 -0.26" rpy="0 0 0"/>
       <geometry>
         <mesh filename="file:///$(find bb8_description)/meshes/head.stl" scale="0.001 0.001 0.001"/>
       </geometry>
-    </collision> -->
+    </collision>
     <xacro:inertial_cylinder mass="0.5" length="0.15" radius="0.15">
         <origin xyz="0 0 0.045" rpy="0 0 0"/>

File: src/bb8_description/urdf/lidar.xacro (robot description, xacro)
@@ -13,9 +13,9 @@
             <material name="black"/>
         </visual>
-        <collision>
+        <!-- <collision>
             <geometry>
                 <cylinder radius="0.05" length="0.04"/>
             </geometry>
-        </collision>
+        </collision> -->
         <inertial>
             <mass value="0.1"/>

File: src/bb8_description/urdf/ros2_control.xacro (robot description, xacro)
@@ -23,6 +23,6 @@
         <joint name="head_x_joint">
             <command_interface name="position">
-                <param name="min">-20</param>
-                <param name="max">20</param>
+                <param name="min">-45</param>
+                <param name="max">45</param>
             </command_interface>
             <state_interface name="position"/>
@@ -30,6 +30,6 @@
         <joint name="head_y_joint">
             <command_interface name="position">
-                <param name="min">-20</param>
-                <param name="max">20</param>
+                <param name="min">-45</param>
+                <param name="max">45</param>
             </command_interface>
             <state_interface name="position"/>

File: src/bb8_description/urdf/sphere.xacro (robot description, xacro)
@@ -28,17 +28,18 @@
   </joint>
   <gazebo reference="sphere_link">
-    <mu>1.0</mu>
-    <mu2>1.0</mu2>
-    <collision>
-      <surface>
-        <contact>
-          <ode>
-            <min_depth>0.001</min_depth>
-          </ode>
-        </contact>
-      </surface>
-      <margin>0.01</margin>
-    </collision>
-   </gazebo>
+    <mu>10</mu>
+    <mu2>10</mu2>
+    <self_collide>false</self_collide>
+    <surface>
+      <contact>
+        <ode>
+          <min_depth>0.01</min_depth>  <!-- Minimum penetration depth for collision response -->
+          <margin>0.01</margin>        <!-- Distance buffer for collision detection -->
+        </ode>
+        <stiffness>1e3</stiffness>     <!-- Contact stiffness -->
+        <damping>1e2</damping>         <!-- Contact damping -->
+      </contact>
+    </surface>
+  </gazebo>
     <gazebo>
       <plugin name="libgazebo_ros_p3d" filename="libgazebo_ros_p3d.so">

File: src/bb8_description/urdf/supports.xacro (robot description, xacro)
@@ -17,5 +17,5 @@
       <collision>
         <geometry>
-          <sphere radius="0.005"/>
+          <sphere radius="0.0049"/>
         </geometry>
       </collision>
@@ -34,28 +34,36 @@
       <parent link="${prefix}_virtual"/>
       <child link="${prefix}_sphere"/>
-      <origin xyz="0.2494 0 0" rpy="0 0 0"/>
+      <origin xyz="0.25 0 0" rpy="0 0 0"/>
     </joint>
     <!-- Physics properties -->
     <gazebo reference="${prefix}_sphere">
-      <mu>0.001</mu>
-      <mu2>0.001</mu2>
+      <mu>1e-6</mu>
+      <mu2>1e-6</mu2>
       <self_collide>true</self_collide>
-      <contact>
-        <collide_without_contact>false</collide_without_contact>
-        <stiffness>1e3</stiffness>
-        <damping>10</damping>
-      </contact>
+      <surface>
+        <contact>
+          <ode>
+            <min_depth>0.01</min_depth>  <!-- Minimum penetration depth for collision response -->
+            <margin>0.01</margin>        <!-- Distance buffer for collision detection -->
+          </ode>
+          <stiffness>1e3</stiffness>     <!-- Contact stiffness -->
+          <damping>1e2</damping>         <!-- Contact damping -->
+        </contact>
+      </surface>
     </gazebo>
   </xacro:macro>
-  <!-- <xacro:spherical_support prefix="support1" angle_1="$(eval pi/4)" angle_2="$(eval 0)"/> -->
-  <!-- <xacro:spherical_support prefix="support2" angle_1="$(eval pi/4)" angle_2="$(eval 4*pi/4)"/> -->
-  <xacro:spherical_support prefix="support1" angle_1="$(eval pi/4)" angle_2="$(eval pi/4)"/>
-  <xacro:spherical_support prefix="support2" angle_1="$(eval pi/4)" angle_2="$(eval 3*pi/4)"/>
-  <xacro:spherical_support prefix="support3" angle_1="$(eval pi/4)" angle_2="$(eval 5*pi/4)"/>
-  <xacro:spherical_support prefix="support4" angle_1="$(eval pi/4)" angle_2="$(eval 7*pi/4)"/>
-  <xacro:spherical_support prefix="support5" angle_1="$(eval -pi/3)" angle_2="$(eval 0)"/>
-  <xacro:spherical_support prefix="support6" angle_1="$(eval -pi/3)" angle_2="$(eval pi/2)"/>
-  <xacro:spherical_support prefix="support7" angle_1="$(eval -pi/3)" angle_2="$(eval pi)"/>
-  <xacro:spherical_support prefix="support8" angle_1="$(eval -pi/3)" angle_2="$(eval 3*pi/2)"/>
+  <!-- <xacro:spherical_support prefix="support1" angle_1="$(eval pi/4)" angle_2="$(eval 0)"/>
+  <xacro:spherical_support prefix="support2" angle_1="$(eval pi/4)" angle_2="$(eval 4*pi/4)"/> -->
+  <!-- <xacro:spherical_support prefix="support3" angle_1="$(eval pi/4)" angle_2="$(eval pi/4)"/>
+  <xacro:spherical_support prefix="support4" angle_1="$(eval pi/4)" angle_2="$(eval 3*pi/4)"/>
+  <xacro:spherical_support prefix="support5" angle_1="$(eval pi/4)" angle_2="$(eval 5*pi/4)"/>
+  <xacro:spherical_support prefix="support6" angle_1="$(eval pi/4)" angle_2="$(eval 7*pi/4)"/> -->
+  <xacro:spherical_support prefix="support7" angle_1="$(eval -pi/3)" angle_2="$(eval 0)"/>
+  <xacro:spherical_support prefix="support8" angle_1="$(eval -pi/3)" angle_2="$(eval 2*pi/3)"/>
+  <xacro:spherical_support prefix="support9" angle_1="$(eval -pi/3)" angle_2="$(eval 4*pi/3)"/>
+  <!-- <xacro:spherical_support prefix="support10" angle_1="$(eval -pi/3)" angle_2="$(eval 0)"/> -->
+  <!-- <xacro:spherical_support prefix="support11" angle_1="$(eval -pi/3)" angle_2="$(eval pi/2)"/> -->
+  <!-- <xacro:spherical_support prefix="support12" angle_1="$(eval -pi/3)" angle_2="$(eval pi)"/> -->
+  <!-- <xacro:spherical_support prefix="support13" angle_1="$(eval -pi/3)" angle_2="$(eval 3*pi/2)"/> -->
   <!-- Connect supports to base -->
   <joint name="supports_joint" type="fixed">
