Commit message: semi-working

File: src/bb8_description/urdf/common_properties.xacro (robot description, xacro)
@@ -3,7 +3,7 @@
   <!-- Constants -->
   <xacro:property name="base_radius" value="0.05" /> <!-- Radius of the circular base -->
-  <xacro:property name="wheel_radius" value="0.03" /> <!-- Radius of the wheels -->
-  <xacro:property name="wheel_separation" value="0.12" /> <!-- Distance between the wheels -->
-  <xacro:property name="sphere_radius" value="0.15" /> <!-- Radius of the outer sphere -->
+  <xacro:property name="wheel_radius" value="0.069" /> <!-- Radius of the wheels -->
+  <xacro:property name="wheel_separation" value="0.364" /> <!-- Distance between the wheels -->
+  <xacro:property name="sphere_radius" value="0.51" /> <!-- Radius of the outer sphere -->
   <!-- Materials -->
   <material name="blue">

File: src/bb8_description/urdf/hamster.xacro (robot description, xacro)
@@ -6,5 +6,6 @@
     <visual>
       <geometry>
-        <cylinder length="0.01" radius="${base_radius}" />
+        <mesh filename="file:///$(find bb8_description)/meshes/frame.stl" scale="0.001 0.001 0.001"/>
+        <!-- <cylinder length="0.01" radius="${base_radius}" /> -->
       </geometry>
       <material name="blue"/>
@@ -12,9 +13,11 @@
     <collision>
       <geometry>
-        <cylinder length="0.01" radius="${base_radius}" />
+        <!-- <mesh filename="file:///$(find bb8_description)/meshes/frame.stl" scale="0.001 0.001 0.0001"/> -->
+        <mesh filename="file:///$(find bb8_description)/meshes/frame.stl" scale="0.000999 0.000999 0.000999"/>
+        <!-- <cylinder length="0.01" radius="${base_radius}" /> -->
       </geometry>
     </collision>
     <inertial>
-      <mass value="0.5"/>
+      <mass value="0.01"/>
       <inertia ixx="0.1" iyy="0.1" izz="0.1" ixy="0.0" ixz="0.0" iyz="0.0"/>
     </inertial>
@@ -23,16 +26,20 @@
   <link name="left_wheel">
     <visual>
+      <origin xyz="${wheel_separation/2 - 0.024} 0 0.1458" rpy="0 0 ${pi}"/>
       <geometry>
-        <cylinder length="0.025" radius="${wheel_radius}" />
+        <mesh filename="file:///$(find bb8_description)/meshes/wheel.stl" scale="0.001 0.001 0.001"/>
+        <!-- <cylinder length="0.025" radius="${wheel_radius}" /> -->
       </geometry>
       <material name="black"/>
     </visual>
     <collision>
+      <origin xyz="${wheel_separation/2 - 0.024} 0 0.1458" rpy="0 0 ${pi}"/>
       <geometry>
-        <cylinder length="0.025" radius="${wheel_radius}" />
+        <mesh filename="file:///$(find bb8_description)/meshes/wheel.stl" scale="0.001 0.001 0.001"/>
+        <!-- <cylinder length="0.025" radius="${wheel_radius}" /> -->
       </geometry>
     </collision>
     <inertial>
-      <mass value="0.1"/>
+      <mass value="0.05"/>
       <inertia ixx="0.01" iyy="0.01" izz="0.01" ixy="0.0" ixz="0.0" iyz="0.0"/>
     </inertial>
@@ -41,16 +48,20 @@
   <link name="right_wheel">
     <visual>
+      <origin xyz="-${wheel_separation/2} 0 0.1458" rpy="0 0 0"/>
       <geometry>
-        <cylinder length="0.025" radius="${wheel_radius}" />
+        <mesh filename="file:///$(find bb8_description)/meshes/wheel.stl" scale="0.001 0.001 0.001"/>
+        <!-- <cylinder length="0.025" radius="${wheel_radius}" /> -->
       </geometry>
       <material name="black"/>
     </visual>
     <collision>
+      <origin xyz="-${wheel_separation/2} 0 0.1458" rpy="0 0 0"/>
       <geometry>
-        <cylinder length="0.025" radius="${wheel_radius}" />
+        <mesh filename="file:///$(find bb8_description)/meshes/wheel.stl" scale="0.001 0.001 0.001"/>
+        <!-- <cylinder length="0.025" radius="${wheel_radius}" /> -->
       </geometry>
     </collision>
     <inertial>
-      <mass value="0.1"/>
+      <mass value="0.05"/>
       <inertia ixx="0.01" iyy="0.01" izz="0.01" ixy="0.0" ixz="0.0" iyz="0.0"/>
     </inertial>
@@ -65,12 +76,12 @@
     <parent link="base_link"/>
     <child link="left_wheel"/>
-    <origin xyz="-${wheel_separation / 2} 0 0" rpy="0 1.57075 0"/>
-    <axis xyz="0 0 1"/>
+    <origin xyz="-${wheel_separation/2} 0 -0.1458" rpy="0 0 ${pi}"/>
+    <axis xyz="-1 0 0"/>
   </joint>
   <joint name="right_wheel_joint" type="continuous">
     <parent link="base_link"/>
     <child link="right_wheel"/>
-    <origin xyz="${wheel_separation / 2} 0 0" rpy="0 1.57075 0"/>
-    <axis xyz="0 0 1"/>
+    <origin xyz="${wheel_separation/2} 0 -0.1458" rpy="0 0 0"/>
+    <axis xyz="1 0 0"/>
   </joint>
   <!-- Gazebo Plugins -->
@@ -92,10 +103,16 @@
   <!-- Collision Tuning for Robot and Sphere -->
   <gazebo reference="left_wheel">
-    <mu>1.0</mu>
-    <mu2>1.0</mu2>
+    <mu>100.0</mu>
+    <mu2>100.0</mu2>
+    <!-- <self_collide>true</self_collide> -->
   </gazebo>
   <gazebo reference="right_wheel">
-    <mu>1.0</mu>
-    <mu2>1.0</mu2>
+    <mu>100.0</mu>
+    <mu2>100.0</mu2>
+    <!-- <self_collide>true</self_collide> -->
+  </gazebo>
+  <gazebo reference="base_link">
+    <mu>0.01</mu>
+    <mu2>0.01</mu2>
   </gazebo>
 </robot>

File: src/bb8_description/urdf/sphere.xacro (robot description, xacro)
@@ -5,5 +5,5 @@
     <visual>
       <geometry>
-        <mesh filename="file:///$(find bb8_description)/meshes/sphere_hollow.stl" scale="0.5 0.5 0.5"/>
+        <mesh filename="file:///$(find bb8_description)/meshes/sphere.stl" scale="0.001 0.001 0.001"/>
       </geometry>
       <material name="white_transparent">
@@ -13,17 +13,9 @@
     <collision>
       <geometry>
-        <mesh filename="file:///$(find bb8_description)/meshes/sphere_hollow.stl" scale="0.5 0.5 0.5"/>
+        <mesh filename="file:///$(find bb8_description)/meshes/sphere.stl" scale="0.001 0.001 0.001"/>
       </geometry>
-      <surface>
-        <friction>
-          <ode>
-            <mu>1.0</mu>
-            <mu2>1.0</mu2>
-          </ode>
-        </friction>
-      </surface>
     </collision>
     <inertial>
-      <mass value="1.0"/>
+      <mass value="1"/>
       <inertia ixx="0.2" iyy="0.2" izz="0.2" ixy="0.0" ixz="0.0" iyz="0.0"/>
     </inertial>
@@ -33,5 +25,6 @@
     <parent link="base_footprint"/>
     <child link="sphere_link"/>
-    <origin xyz="0 0 ${sphere_radius}" rpy="0 0 0"/>
+    <origin xyz="0 0 0" rpy="0 0 0"/>
+    <!-- <origin xyz="0 0 ${sphere_radius}" rpy="0 0 0"/> -->
   </joint>
   <gazebo>

Commit message: cleanup

File: src/bb8_description/urdf/common_properties.xacro (robot description, xacro)
@@ -2,5 +2,4 @@
 <robot xmlns:xacro="http://www.ros.org/wiki/xacro">
   <!-- Constants -->
-  <xacro:property name="base_radius" value="0.05" /> <!-- Radius of the circular base -->
   <xacro:property name="wheel_radius" value="0.069" /> <!-- Radius of the wheels -->
   <xacro:property name="wheel_separation" value="0.3641" /> <!-- Distance between the wheels -->
@@ -39,5 +38,5 @@
   </material>
   <gazebo reference="base_link">
-  <material>Gazebo/Blue</material>
+    <material>Gazebo/Blue</material>
   </gazebo>
   <gazebo reference="left_wheel">

File: src/bb8_description/urdf/gazebo_plugins.xacro (robot description, xacro)
@@ -1,13 +1,4 @@
 <?xml version="1.0"?>
 <robot xmlns:xacro="http://www.ros.org/wiki/xacro">
-  <!-- <gazebo>
-    <plugin name="gazebo_ros_joint_state_publisher" filename="libgazebo_ros_joint_state_publisher.so">
-      <joint_name>right_wheel_joint</joint_name>
-      <joint_name>left_wheel_joint</joint_name>
-      <joint_name>head_x_joint</joint_name>
-      <joint_name>head_y_joint</joint_name>
-      <update_rate>100.0</update_rate>
-    </plugin>
-  </gazebo> -->
   <gazebo>
     <plugin name="libgazebo_ros_p3d" filename="libgazebo_ros_p3d.so">

Commit message: Removed unnecessary stuff. Trying new approach for driving inside sphere

File: src/bb8_description/urdf/common_properties.xacro (robot description, xacro)
@@ -2,7 +2,9 @@
 <robot xmlns:xacro="http://www.ros.org/wiki/xacro">
   <!-- Constants -->
-  <xacro:property name="wheel_radius" value="0.069" /> <!-- Radius of the wheels -->
-  <xacro:property name="wheel_separation" value="0.3641" /> <!-- Distance between the wheels -->
-  <xacro:property name="sphere_radius" value="0.51" /> <!-- Radius of the outer sphere -->
+  <xacro:property name="wheel_radius" value="0.069" /> <!-- Radius of the wheels contact -->
+  <xacro:property name="wheel_contact_separation" value="0.3641" /> <!-- Distance between the wheels contact points-->
+  <xacro:property name="wheel_separation" value="0.3437" /> <!-- Distance between the wheels -->
+  <xacro:property name="sphere_radius_o" value="0.26" /> <!-- Outer sphere radius -->
+  <xacro:property name="sphere_radius_i" value="0.255" /> <!-- Inner sphere radius -->
   <!-- Inertia -->
   <xacro:macro name="inertial_sphere" params="mass radius *origin">

File: src/bb8_description/urdf/hamster.xacro (robot description, xacro)
@@ -2,9 +2,13 @@
 <robot xmlns:xacro="http://www.ros.org/wiki/xacro">
   <!-- Base Footprint -->
+  <!-- This frame is always at the fround, represents robot position and orientation in 2d -->
   <link name="base_footprint" />
+  <link name="sphere_center" />
+  <!-- <link name="base_roll" /> -->
+  <!-- <link name="base_pitch" /> -->
   <!-- Base Link -->
   <link name="base_link">
     <visual>
-      <origin xyz="0 0 -${0.1458 + 0.025}" rpy="0 0 0"/>
+      <origin xyz="0 0 0" rpy="0 0 0"/>
       <geometry>
         <cylinder length="0.05" radius="0.09" />
@@ -13,5 +17,5 @@
     </visual>
     <xacro:inertial_cylinder mass="0.5" length="0.05" radius="0.09">
-      <origin xyz="0 0 -${0.1458 + 0.025}" rpy="0 0 0"/>
+      <origin xyz="0 0 0" rpy="0 0 0"/>
     </xacro:inertial_cylinder>
   </link>
@@ -31,5 +35,5 @@
   <link name="left_wheel">
     <visual>
-      <origin xyz="0 0 0" rpy="0 ${pi/2} 0"/>
+      <origin xyz="0 0 0" rpy="${pi/2} 0 0"/>
       <geometry>
         <mesh filename="file:///$(find bb8_description)/meshes/wheel.stl" scale="0.001 0.001 0.001"/>
@@ -38,5 +42,5 @@
     </visual>
     <collision>
-      <origin xyz="0 0 0" rpy="0 ${pi/2} 0"/>
+      <origin xyz="0 0 0" rpy="${pi/2} 0 0"/>
       <geometry>
         <mesh filename="file:///$(find bb8_description)/meshes/wheel.stl" scale="0.001 0.001 0.001"/>
@@ -44,22 +48,11 @@
     </collision>
     <xacro:inertial_sphere mass="0.05" radius="0.076">
-      <origin xyz="0 0 0" rpy="0 ${pi/2} 0"/>
+      <origin xyz="0 0 0" rpy="${pi/2} 0 0"/>
     </xacro:inertial_sphere>
-  </link>
-  <link name="wheel_connector" >
-    <visual>
-      <geometry>
-        <cylinder length="0.01" radius="0.01" />
-      </geometry>
-      <material name="blue"/>
-    </visual>
-    <xacro:inertial_cylinder mass="0.01" length="0.01" radius="0.01">
-      <origin xyz="0 0 0" rpy="0 0 0"/>
-    </xacro:inertial_cylinder>
   </link>
   <!-- Right Wheel -->
   <link name="right_wheel">
     <visual>
-      <origin xyz="0 0 0" rpy="0 ${pi/2} 0"/>
+      <origin xyz="0 0 0" rpy="${pi/2} 0 0"/>
       <geometry>
         <mesh filename="file:///$(find bb8_description)/meshes/wheel.stl" scale="0.001 0.001 0.001"/>
@@ -68,5 +61,5 @@
     </visual>
     <collision>
-      <origin xyz="0 0 0" rpy="0 ${pi/2} 0"/>
+      <origin xyz="0 0 0" rpy="${pi/2} 0 0"/>
       <geometry>
         <mesh filename="file:///$(find bb8_description)/meshes/wheel.stl" scale="0.001 0.001 0.001"/>
@@ -74,37 +67,34 @@
     </collision>
     <xacro:inertial_sphere mass="0.05" radius="0.076">
-      <origin xyz="0 0 0" rpy="0 ${pi/2} 0"/>
+      <origin xyz="0 0 0" rpy="${pi/2} 0 0"/>
     </xacro:inertial_sphere>
   </link>
   <!-- Joints -->
+  <joint name="base_footprint_joint" type="fixed">
+    <parent link="base_footprint" />
+    <child link="sphere_center" />
+    <origin xyz="0 0 ${sphere_radius_o}" rpy="0 0 0"/>
+  </joint>
   <joint name="base_joint" type="fixed">
-  <!-- It should be floating, but for some reason it does not work with it -->
-  <!-- Anyway, it would be converted to fixed when loading urdf to gazebo -->
-  <!-- <joint name="base_joint" type="floating"> -->
-    <parent link="base_footprint" />
+    <parent link="sphere_center" />
     <child link="base_link" />
-    <origin xyz="0 0 0" rpy="0 0 0"/>
-  </joint>
-  <joint name="wheel_connector_joint" type="fixed">
-    <parent link="base_link" />
-    <child link="wheel_connector" />
-    <origin xyz="0 0 0" rpy="0 0 ${pi/2}"/>
+    <origin xyz="0 0 -0.1458" rpy="0 0 0"/>
   </joint>
   <joint name="counterweight_joint" type="fixed">
     <parent link="base_link" />
     <child link="counterweight" />
-    <origin xyz="0 0 -0.21" rpy="0 0 0"/>
+    <origin xyz="0 0 -0.03" rpy="0 0 0"/>
   </joint>
   <joint name="left_wheel_joint" type="continuous">
-    <parent link="wheel_connector"/>
+    <parent link="base_link"/>
     <child link="left_wheel"/>
-    <origin xyz="${0.3437/2} 0 -0.1458" rpy="0 0 0"/>
-    <axis xyz="1 0 0"/>
+    <origin xyz="0 ${wheel_separation/2}  0" rpy="0 0 0"/>
+    <axis xyz="0 1 0"/>
   </joint>
   <joint name="right_wheel_joint" type="continuous">
-    <parent link="wheel_connector"/>
+    <parent link="base_link"/>
     <child link="right_wheel"/>
-    <origin xyz="-${0.3437/2} 0 -0.1458" rpy="0 0 0"/>
-    <axis xyz="1 0 0"/>
+    <origin xyz="0 -${wheel_separation/2} 0" rpy="0 0 0"/>
+    <axis xyz="0 1 0"/>
   </joint>
   <!-- Collision Tuning for Robot and Sphere -->

File: src/bb8_description/urdf/head.xacro (robot description, xacro)
@@ -36,5 +36,5 @@
   <!-- Revolute joints with limits for full ball joint motion -->
   <joint name="head_x_joint" type="revolute">
-    <parent link="base_link"/>
+    <parent link="sphere_center"/>
     <child link="head_x_link"/>
     <origin xyz="0 0 0" rpy="0 0 0"/>

File: src/bb8_description/urdf/sensors.xacro (robot description, xacro)
@@ -4,5 +4,11 @@
   <xacro:macro name="imu_sensor" params="parent_link sensor_name">
     <!-- IMU Link -->
-    <link name="${sensor_name}_link" />
+    <link name="${sensor_name}_link" >
+      <visual>
+      <geometry>
+        <cylinder length="0.01" radius="0.01" />
+      </geometry>
+      </visual>
+    </link>
     <!-- IMU Joint -->
     <joint name="${sensor_name}_joint" type="fixed">
@@ -42,5 +48,5 @@
     </gazebo>
   </xacro:macro>
-  <xacro:imu_sensor parent_link="base_link" sensor_name="imu_base"/>
+  <xacro:imu_sensor parent_link="sphere_center" sensor_name="imu_base"/>
   <!-- <xacro:imu_sensor parent_link="head" sensor_name="imu_head"/> -->
 </robot>

File: src/bb8_description/urdf/sphere.xacro (robot description, xacro)
@@ -5,5 +5,5 @@
     <visual>
       <geometry>
-        <mesh filename="file:///$(find bb8_description)/meshes/sphere.stl" scale="0.001 0.001 0.001"/>
+        <mesh filename="file:///$(find bb8_description)/meshes/sphere.stl"/>
       </geometry>
       <material name="white_transparent">
@@ -13,5 +13,5 @@
     <collision>
       <geometry>
-        <mesh filename="file:///$(find bb8_description)/meshes/sphere.stl" scale="0.001 0.001 0.001"/>
+        <mesh filename="file:///$(find bb8_description)/meshes/sphere.stl"/>
       </geometry>
     </collision>
@@ -23,33 +23,21 @@
   <!-- Joint to Connect Sphere and Hamster -->
   <joint name="sphere_joint" type="floating">
-    <parent link="base_footprint"/>
+    <parent link="sphere_center"/>
     <child link="sphere_link"/>
-    <origin rpy="0 0 0" xyz="0 0 0"/>
   </joint>
   <gazebo reference="sphere_link">
-    <mu>10</mu>
-    <mu2>10</mu2>
+    <mu>10.0</mu>
+    <mu2>10.0</mu2>
     <self_collide>false</self_collide>
     <surface>
       <contact>
         <ode>
-          <min_depth>0.001</min_depth>
-          <margin>0.001</margin>
+          <min_depth>1</min_depth>
+          <margin>1</margin>
         </ode>
-        <stiffness>1e5</stiffness>     <!-- Contact stiffness -->
-        <damping>1e3</damping>         <!-- Contact damping -->
+        <stiffness>1e-10</stiffness>
+        <damping>1e10</damping>
       </contact>
     </surface>
   </gazebo>
-    <gazebo>
-      <plugin name="libgazebo_ros_p3d" filename="libgazebo_ros_p3d.so">
-      <ros>
-        <remapping>odom:=sphere_pose</remapping>
-      </ros>
-      <frame_name>base_footprint</frame_name>
-      <body_name>sphere_link</body_name>
-      <update_rate>50</update_rate>
-      <gaussian_noise>0.01</gaussian_noise>
-      </plugin>
-    </gazebo>
 </robot>

File: src/bb8_description/urdf/supports.xacro (robot description, xacro)
@@ -34,19 +34,19 @@
       <parent link="${prefix}_virtual"/>
       <child link="${prefix}_sphere"/>
-      <origin xyz="0.249 0 0" rpy="0 0 0"/>
+      <origin xyz="0.25 0 0" rpy="0 0 0"/>
     </joint>
     <!-- Physics properties -->
     <gazebo reference="${prefix}_sphere">
-      <mu>1e-6</mu>
-      <mu2>1e-6</mu2>
+      <mu>0</mu>
+      <mu2>0</mu2>
       <self_collide>true</self_collide>
       <surface>
         <contact>
           <ode>
-            <min_depth>0.01</min_depth>  <!-- Minimum penetration depth for collision response -->
-            <margin>0.01</margin>        <!-- Distance buffer for collision detection -->
+            <min_depth>1</min_depth>  <!-- Minimum penetration depth for collision response -->
+            <margin>1</margin>        <!-- Distance buffer for collision detection -->
           </ode>
-          <stiffness>1e6</stiffness>     <!-- Contact stiffness -->
-          <damping>1e4</damping>         <!-- Contact damping -->
+          <stiffness>1e-10</stiffness>     <!-- Contact stiffness -->
+          <damping>1e10</damping>         <!-- Contact damping -->
         </contact>
       </surface>
@@ -54,20 +54,8 @@
     </gazebo>
   </xacro:macro>
-  <!-- <xacro:spherical_support prefix="support1" angle_1="$(eval pi/4)" angle_2="$(eval 0)"/>
-  <xacro:spherical_support prefix="support2" angle_1="$(eval pi/4)" angle_2="$(eval 4*pi/4)"/> -->
-  <!-- <xacro:spherical_support prefix="support3" angle_1="$(eval pi/4)" angle_2="$(eval pi/4)"/>
-  <xacro:spherical_support prefix="support4" angle_1="$(eval pi/4)" angle_2="$(eval 3*pi/4)"/>
-  <xacro:spherical_support prefix="support5" angle_1="$(eval pi/4)" angle_2="$(eval 5*pi/4)"/>
-  <xacro:spherical_support prefix="support6" angle_1="$(eval pi/4)" angle_2="$(eval 7*pi/4)"/> -->
-  <xacro:spherical_support prefix="support7" angle_1="$(eval -pi/3)" angle_2="$(eval 0)"/>
-  <xacro:spherical_support prefix="support8" angle_1="$(eval -pi/3)" angle_2="$(eval 2*pi/3)"/>
-  <xacro:spherical_support prefix="support9" angle_1="$(eval -pi/3)" angle_2="$(eval 4*pi/3)"/>
-  <xacro:spherical_support prefix="support10" angle_1="$(eval -pi/3)" angle_2="$(eval 0)"/>
-  <xacro:spherical_support prefix="support11" angle_1="$(eval -pi/3)" angle_2="$(eval pi/2)"/>
-  <xacro:spherical_support prefix="support12" angle_1="$(eval -pi/3)" angle_2="$(eval pi)"/>
-  <xacro:spherical_support prefix="support13" angle_1="$(eval -pi/3)" angle_2="$(eval 3*pi/2)"/>
+  <xacro:spherical_support prefix="support1" angle_1="$(eval -pi/2)" angle_2="$(eval 0)"/>
   <!-- Connect supports to base -->
   <joint name="supports_joint" type="fixed">
-    <parent link="base_link"/>
+    <parent link="sphere_center"/>
     <child link="supports"/>
     <origin xyz="0 0 0" rpy="0 0 0"/>
