Commit message: added head

File: src/bb8_description/urdf/hamster.xacro (robot description, xacro)
@@ -7,26 +7,13 @@
       <origin xyz="0 0 -${0.1458 + 0.025}" rpy="0 0 0"/>
       <geometry>
-        <!-- <mesh filename="file:///$(find bb8_description)/meshes/frame_b.stl" scale="0.000995 0.000995 0.000995"/> -->
         <cylinder length="0.05" radius="0.09" />
       </geometry>
       <material name="blue"/>
     </visual>
-    <!-- No need for collision -->
-    <!-- <collision>
-      <geometry>
-        <mesh filename="file:///$(find bb8_description)/meshes/frame_b.stl" scale="0.000995 0.000995 0.000995"/>
-      </geometry>
-    </collision> -->
-    <inertial>
-      <mass value="0.5"/>
-      <inertia ixx="0.1" iyy="0.1" izz="0.1" ixy="0.0" ixz="0.0" iyz="0.0"/>
-    </inertial>
   </link>
   <link name="counterweight">
     <visual>
-      <!-- STL origin is messed up, so need to move it -->
-      <origin xyz="0 0 ${0.19+0.05}" rpy="0 0 0"/>
       <geometry>
-        <mesh filename="file:///$(find bb8_description)/meshes/counterweight.stl" scale="0.001 0.001 0.001"/>
+        <cylinder length="0.04" radius="0.07" />
       </geometry>
       <material name="black"/>
@@ -82,5 +69,5 @@
       <parent link="base_link" />
       <child link="counterweight" />
-      <origin xyz="0 0 -${0.19+0.05}" rpy="0 0 0"/>
+      <origin xyz="0 0 -0.21" rpy="0 0 0"/>
   </joint>
   <joint name="left_wheel_joint" type="continuous">
@@ -114,4 +101,5 @@
   <!-- Collision Tuning for Robot and Sphere -->
   <gazebo reference="left_wheel">
+    <self_collide>true</self_collide>
     <surface>
       <contact>
@@ -129,4 +117,5 @@
   </gazebo>
   <gazebo reference="right_wheel">
+    <self_collide>true</self_collide>
     <surface>
       <contact>

File: src/bb8_description/urdf/head.xacro (robot description, xacro)
@@ -3,4 +3,5 @@
   <link name="head">
     <visual>
+      <origin xyz="0 0 -0.26" rpy="0 0 0"/>
       <geometry>
         <mesh filename="file:///$(find bb8_description)/meshes/head.stl" scale="0.001 0.001 0.001"/>
@@ -11,4 +12,5 @@
     </visual>
     <collision>
+      <origin xyz="0 0 -0.26" rpy="0 0 0"/>
       <geometry>
         <mesh filename="file:///$(find bb8_description)/meshes/head.stl" scale="0.001 0.001 0.001"/>
@@ -16,12 +18,50 @@
     </collision>
     <inertial>
-      <mass value="1.5"/>
-      <inertia ixx="0.4" iyy="0.4" izz="0.4" ixy="0.0" ixz="0.0" iyz="0.0"/>
+      <mass value="1.0"/>
+      <inertia ixx="0.2" iyy="0.2" izz="0.2" ixy="0.0" ixz="0.0" iyz="0.0"/>
     </inertial>
   </link>
-  <joint name="head_joint" type="fixed">
+  <!-- Intermediate links for ball joint -->
+  <link name="head_x_link">
+    <inertial>
+      <mass value="0.01"/>
+      <inertia ixx="0.001" iyy="0.001" izz="0.001" ixy="0.0" ixz="0.0" iyz="0.0"/>
+    </inertial>
+  </link>
+  <link name="head_y_link">
+    <inertial>
+      <mass value="0.01"/>
+      <inertia ixx="0.001" iyy="0.001" izz="0.001" ixy="0.0" ixz="0.0" iyz="0.0"/>
+    </inertial>
+  </link>
+  <!-- Revolute joints with limits for full ball joint motion -->
+  <joint name="head_x_joint" type="revolute">
     <parent link="base_link"/>
+    <child link="head_x_link"/>
+    <origin xyz="0 0 0" rpy="0 0 0"/>
+    <axis xyz="1 0 0"/>
+    <limit lower="-${pi/9}" upper="${pi/9}" effort="10" velocity="1.0"/>
+    <dynamics damping="0.1" friction="0.01"/>
+  </joint>
+  <joint name="head_y_joint" type="revolute">
+    <parent link="head_x_link"/>
+    <child link="head_y_link"/>
+    <origin xyz="0 0 0" rpy="0 0 0"/>
+    <axis xyz="0 1 0"/>
+    <limit lower="-${pi/9}" upper="${pi/9}" effort="10" velocity="1.0"/>
+    <dynamics damping="0.1" friction="0.01"/>
+  </joint>
+  <!-- Fixed joint to attach head to the final rotation link -->
+  <joint name="head_attachment" type="fixed">
+    <parent link="head_y_link"/>
     <child link="head"/>
-    <origin xyz="0 0 0" rpy="0 0 0"/>
+    <origin xyz="0 0 0.26" rpy="0 0 0"/>
   </joint>
+  <gazebo>
+    <plugin name="gazebo_ros_joint_state_publisher" filename="libgazebo_ros_joint_state_publisher.so">
+      <joint_name>head_x_joint</joint_name>
+      <joint_name>head_y_joint</joint_name>
+      <update_rate>100.0</update_rate>
+    </plugin>
+  </gazebo>
 </robot>

File: src/bb8_description/urdf/sphere.xacro (robot description, xacro)
@@ -41,5 +41,4 @@
     <mu>0.5</mu>
     <mu2>0.5</mu2>
-    <self_collide>true</self_collide>
     <collision>
       <margin>0.01</margin>

File: src/bb8_description/urdf/supports.xacro (robot description, xacro)
@@ -40,4 +40,5 @@
       <mu>0.01</mu>
       <mu2>0.01</mu2>
+      <self_collide>true</self_collide>
       <contact>
         <collide_without_contact>false</collide_without_contact>

Commit message: changed base_footprint position, added transform publisher for floating joint between base_footprint and base_link

File: src/bb8_description/urdf/hamster.xacro (robot description, xacro)
@@ -78,8 +78,8 @@
   </link>
   <!-- Joints -->
-  <joint name="base_joint" type="fixed">
+  <joint name="base_joint" type="floating">
     <parent link="base_footprint" />
     <child link="base_link" />
-    <origin xyz="0 0 0" rpy="0 0 0"/>
+    <origin xyz="0 0 0.25" rpy="0 0 0"/>
   </joint>
   <joint name="wheel_connector_joint" type="fixed">

File: src/bb8_description/urdf/sensors.xacro (robot description, xacro)
@@ -43,4 +43,4 @@
   </xacro:macro>
   <xacro:imu_sensor parent_link="base_link" sensor_name="imu_base"/>
-  <xacro:imu_sensor parent_link="head" sensor_name="imu_head"/>
+  <!-- <xacro:imu_sensor parent_link="head" sensor_name="imu_head"/> -->
 </robot>

File: src/bb8_description/urdf/sphere.xacro (robot description, xacro)
@@ -25,13 +25,6 @@
     <parent link="base_footprint"/>
     <child link="sphere_link"/>
-    <origin xyz="0 0 0" rpy="0 0 0"/>
+    <origin rpy="0 0 0" xyz="0 0 0.26"/>
   </joint>
-  <!-- <gazebo reference="sphere_link">
-    <mu>0.5</mu>
-    <mu2>0.5</mu2>
-    <collision>
-      <margin>0.01</margin>
-    </collision>
-  </gazebo> -->
   <gazebo reference="sphere_link">
     <mu>1.0</mu>
@@ -42,5 +35,5 @@
           <ode>
             <min_depth>0.001</min_depth>
-            </ode>
+          </ode>
         </contact>
       </surface>

Commit message: fixedd a lot of stuff, but now odometry is broken :)

File: src/bb8_description/urdf/hamster.xacro (robot description, xacro)
@@ -78,8 +78,11 @@
   </link>
   <!-- Joints -->
-  <joint name="base_joint" type="floating">
+  <joint name="base_joint" type="fixed">
+  <!-- It should be floating, but for some reason it does not work with it -->
+  <!-- Anyway, it would be converted to fixed when loading urdf to gazebo -->
+  <!-- <joint name="base_joint" type="floating"> -->
     <parent link="base_footprint" />
     <child link="base_link" />
-    <origin xyz="0 0 0.25" rpy="0 0 0"/>
+    <origin xyz="0 0 0" rpy="0 0 0"/>
   </joint>
   <joint name="wheel_connector_joint" type="fixed">

File: src/bb8_description/urdf/sphere.xacro (robot description, xacro)
@@ -25,5 +25,5 @@
     <parent link="base_footprint"/>
     <child link="sphere_link"/>
-    <origin rpy="0 0 0" xyz="0 0 0.26"/>
+    <origin rpy="0 0 0" xyz="0 0 0"/>
   </joint>
   <gazebo reference="sphere_link">
@@ -41,14 +41,14 @@
     </collision>
    </gazebo>
-  <gazebo>
-    <plugin name="libgazebo_ros_p3d" filename="libgazebo_ros_p3d.so">
-    <ros>
-      <remapping>odom:=sphere_pose</remapping>
-    </ros>
-    <frame_name>base_footprint</frame_name>
-    <body_name>sphere_link</body_name>
-    <update_rate>50</update_rate>
-    <gaussian_noise>0.01</gaussian_noise>
-    </plugin>
-  </gazebo>
+    <gazebo>
+      <plugin name="libgazebo_ros_p3d" filename="libgazebo_ros_p3d.so">
+      <ros>
+        <remapping>odom:=sphere_pose</remapping>
+      </ros>
+      <frame_name>base_footprint</frame_name>
+      <body_name>sphere_link</body_name>
+      <update_rate>50</update_rate>
+      <gaussian_noise>0.01</gaussian_noise>
+      </plugin>
+    </gazebo>
 </robot>

File: src/bb8_description/urdf/supports.xacro (robot description, xacro)
@@ -48,13 +48,14 @@
     </gazebo>
   </xacro:macro>
-  <xacro:spherical_support prefix="support1" angle_1="$(eval pi/4)" angle_2="$(eval 0)"/>
-  <xacro:spherical_support prefix="support2" angle_1="$(eval pi/4)" angle_2="$(eval 4*pi/4)"/>
-  <!-- <xacro:spherical_support prefix="support1" angle_1="$(eval pi/4)" angle_2="$(eval pi/4)"/> -->
-  <!-- <xacro:spherical_support prefix="support2" angle_1="$(eval pi/4)" angle_2="$(eval 3*pi/4)"/> -->
-  <!-- <xacro:spherical_support prefix="support6" angle_1="$(eval pi/4)" angle_2="$(eval 5*pi/4)"/> -->
-  <!-- <xacro:spherical_support prefix="support7" angle_1="$(eval pi/4)" angle_2="$(eval 7*pi/4)"/> -->
-  <xacro:spherical_support prefix="support3" angle_1="$(eval -pi/3)" angle_2="$(eval 0)"/>
-  <xacro:spherical_support prefix="support4" angle_1="$(eval -pi/3)" angle_2="$(eval 2*pi/3)"/>
-  <xacro:spherical_support prefix="support5" angle_1="$(eval -pi/3)" angle_2="$(eval 4*pi/3)"/>
+  <!-- <xacro:spherical_support prefix="support1" angle_1="$(eval pi/4)" angle_2="$(eval 0)"/> -->
+  <!-- <xacro:spherical_support prefix="support2" angle_1="$(eval pi/4)" angle_2="$(eval 4*pi/4)"/> -->
+  <xacro:spherical_support prefix="support1" angle_1="$(eval pi/4)" angle_2="$(eval pi/4)"/>
+  <xacro:spherical_support prefix="support2" angle_1="$(eval pi/4)" angle_2="$(eval 3*pi/4)"/>
+  <xacro:spherical_support prefix="support3" angle_1="$(eval pi/4)" angle_2="$(eval 5*pi/4)"/>
+  <xacro:spherical_support prefix="support4" angle_1="$(eval pi/4)" angle_2="$(eval 7*pi/4)"/>
+  <xacro:spherical_support prefix="support5" angle_1="$(eval -pi/3)" angle_2="$(eval 0)"/>
+  <xacro:spherical_support prefix="support6" angle_1="$(eval -pi/3)" angle_2="$(eval pi/2)"/>
+  <xacro:spherical_support prefix="support7" angle_1="$(eval -pi/3)" angle_2="$(eval pi)"/>
+  <xacro:spherical_support prefix="support8" angle_1="$(eval -pi/3)" angle_2="$(eval 3*pi/2)"/>
   <!-- Connect supports to base -->
   <joint name="supports_joint" type="fixed">

Commit message: tried building a map

File: src/bb8_description/urdf/hamster.xacro (robot description, xacro)
@@ -113,4 +113,8 @@
     <surface>
       <contact>
+        <ode>
+          <min_depth>0.05</min_depth>
+          <margin>0.05</margin>
+        </ode>
         <collide_without_contact>false</collide_without_contact>
         <stiffness>1e6</stiffness>
@@ -129,4 +133,8 @@
     <surface>
       <contact>
+        <ode>
+          <min_depth>0.05</min_depth>
+          <margin>0.05</margin>
+        </ode>
         <collide_without_contact>false</collide_without_contact>
         <stiffness>1e6</stiffness>

File: src/bb8_description/urdf/head.xacro (robot description, xacro)
@@ -11,10 +11,10 @@
       </material>
     </visual>
-    <collision>
+    <!-- <collision>
       <origin xyz="0 0 -0.26" rpy="0 0 0"/>
       <geometry>
         <mesh filename="file:///$(find bb8_description)/meshes/head.stl" scale="0.001 0.001 0.001"/>
       </geometry>
-    </collision>
+    </collision> -->
     <xacro:inertial_cylinder mass="0.5" length="0.15" radius="0.15">
         <origin xyz="0 0 0.045" rpy="0 0 0"/>

File: src/bb8_description/urdf/sphere.xacro (robot description, xacro)
@@ -34,6 +34,6 @@
       <contact>
         <ode>
-          <min_depth>0.01</min_depth>  <!-- Minimum penetration depth for collision response -->
-          <margin>0.01</margin>        <!-- Distance buffer for collision detection -->
+          <min_depth>0.01</min_depth>
+          <margin>0.02</margin>
         </ode>
         <stiffness>1e3</stiffness>     <!-- Contact stiffness -->

File: src/bb8_description/urdf/supports.xacro (robot description, xacro)
@@ -17,5 +17,5 @@
       <collision>
         <geometry>
-          <sphere radius="0.0049"/>
+          <sphere radius="0.005"/>
         </geometry>
       </collision>
@@ -34,5 +34,5 @@
       <parent link="${prefix}_virtual"/>
       <child link="${prefix}_sphere"/>
-      <origin xyz="0.25 0 0" rpy="0 0 0"/>
+      <origin xyz="0.2494 0 0" rpy="0 0 0"/>
     </joint>
     <!-- Physics properties -->
@@ -45,18 +45,18 @@
           <ode>
             <min_depth>0.01</min_depth>  <!-- Minimum penetration depth for collision response -->
-            <margin>0.01</margin>        <!-- Distance buffer for collision detection -->
+            <margin>0.02</margin>        <!-- Distance buffer for collision detection -->
           </ode>
-          <stiffness>1e3</stiffness>     <!-- Contact stiffness -->
-          <damping>1e2</damping>         <!-- Contact damping -->
+          <stiffness>1e6</stiffness>     <!-- Contact stiffness -->
+          <damping>1e4</damping>         <!-- Contact damping -->
         </contact>
       </surface>
     </gazebo>
   </xacro:macro>
-  <!-- <xacro:spherical_support prefix="support1" angle_1="$(eval pi/4)" angle_2="$(eval 0)"/>
-  <xacro:spherical_support prefix="support2" angle_1="$(eval pi/4)" angle_2="$(eval 4*pi/4)"/> -->
-  <!-- <xacro:spherical_support prefix="support3" angle_1="$(eval pi/4)" angle_2="$(eval pi/4)"/>
+  <!-- <xacro:spherical_support prefix="support1" angle_1="$(eval pi/4)" angle_2="$(eval 0)"/> -->
+  <!-- <xacro:spherical_support prefix="support2" angle_1="$(eval pi/4)" angle_2="$(eval 4*pi/4)"/> -->
+  <xacro:spherical_support prefix="support3" angle_1="$(eval pi/4)" angle_2="$(eval pi/4)"/>
   <xacro:spherical_support prefix="support4" angle_1="$(eval pi/4)" angle_2="$(eval 3*pi/4)"/>
   <xacro:spherical_support prefix="support5" angle_1="$(eval pi/4)" angle_2="$(eval 5*pi/4)"/>
-  <xacro:spherical_support prefix="support6" angle_1="$(eval pi/4)" angle_2="$(eval 7*pi/4)"/> -->
+  <xacro:spherical_support prefix="support6" angle_1="$(eval pi/4)" angle_2="$(eval 7*pi/4)"/>
   <xacro:spherical_support prefix="support7" angle_1="$(eval -pi/3)" angle_2="$(eval 0)"/>
   <xacro:spherical_support prefix="support8" angle_1="$(eval -pi/3)" angle_2="$(eval 2*pi/3)"/>

Commit message: .

File: src/bb8_description/urdf/hamster.xacro (robot description, xacro)
@@ -35,5 +35,5 @@
       <origin xyz="0 0 0" rpy="${pi/2} 0 0"/>
       <geometry>
-        <mesh filename="file:///$(find bb8_description)/meshes/wheel.stl" scale="0.001 0.001 0.001"/>
+        <mesh filename="file:///$(find bb8_description)/meshes/wheel.stl" />
       </geometry>
       <material name="black"/>
@@ -42,5 +42,5 @@
       <origin xyz="0 0 0" rpy="${pi/2} 0 0"/>
       <geometry>
-        <mesh filename="file:///$(find bb8_description)/meshes/wheel.stl" scale="0.001 0.001 0.001"/>
+        <mesh filename="file:///$(find bb8_description)/meshes/wheel.stl" />
       </geometry>
     </collision>
@@ -54,5 +54,5 @@
       <origin xyz="0 0 0" rpy="${pi/2} 0 0"/>
       <geometry>
-        <mesh filename="file:///$(find bb8_description)/meshes/wheel.stl" scale="0.001 0.001 0.001"/>
+        <mesh filename="file:///$(find bb8_description)/meshes/wheel.stl" />
       </geometry>
       <material name="black"/>
@@ -61,5 +61,5 @@
       <origin xyz="0 0 0" rpy="${pi/2} 0 0"/>
       <geometry>
-        <mesh filename="file:///$(find bb8_description)/meshes/wheel.stl" scale="0.001 0.001 0.001"/>
+        <mesh filename="file:///$(find bb8_description)/meshes/wheel.stl" />
       </geometry>
     </collision>

File: src/bb8_description/urdf/head.xacro (robot description, xacro)
@@ -11,10 +11,10 @@
       </material>
     </visual>
-    <!-- <collision>
+    <collision>
       <origin xyz="0 0 -0.26" rpy="0 0 0"/>
       <geometry>
         <mesh filename="file:///$(find bb8_description)/meshes/head.stl" scale="0.001 0.001 0.001"/>
       </geometry>
-    </collision> -->
+    </collision>
     <xacro:inertial_cylinder mass="0.5" length="0.15" radius="0.15">
         <origin xyz="0 0 0.045" rpy="0 0 0"/>

File: src/bb8_description/urdf/lidar.xacro (robot description, xacro)
@@ -13,9 +13,4 @@
             <material name="black"/>
         </visual>
-        <!-- <collision>
-            <geometry>
-                <cylinder radius="0.05" length="0.04"/>
-            </geometry>
-        </collision> -->
         <inertial>
             <mass value="0.1"/>

File: src/bb8_description/urdf/sphere.xacro (robot description, xacro)
@@ -2,5 +2,5 @@
 <robot xmlns:xacro="http://www.ros.org/wiki/xacro">
   <!-- Dummy links for rotational joints -->
-  <link name="link_yaw">
+  <link name="sphere_yaw">
     <inertial>
       <mass value="0.001"/>
@@ -8,5 +8,5 @@
     </inertial>
   </link>
-  <link name="link_pitch">
+  <link name="sphere_pitch">
     <inertial>
       <mass value="0.001"/>
@@ -14,6 +14,6 @@
     </inertial>
   </link>
-  <!-- Outer Sphere Link -->
-  <link name="sphere_link">
+  <!-- Sphere Shell Link -->
+  <link name="sphere">
     <visual>
       <geometry>
@@ -35,23 +35,23 @@
   </link>
   <!-- Continuous joints -->
-  <joint name="yaw_joint" type="continuous">
+  <joint name="sphere_yaw_joint" type="continuous">
     <parent link="sphere_center"/>
-    <child link="link_yaw"/>
+    <child link="sphere_yaw"/>
     <axis xyz="0 0 1"/>
     <origin xyz="0 0 0" rpy="0 0 0"/>
   </joint>
-  <joint name="pitch_joint" type="continuous">
-    <parent link="link_yaw"/>
-    <child link="link_pitch"/>
+  <joint name="sphere_pitch_joint" type="continuous">
+    <parent link="sphere_yaw"/>
+    <child link="sphere_pitch"/>
     <axis xyz="0 1 0"/>
     <origin xyz="0 0 0" rpy="0 0 0"/>
   </joint>
-  <joint name="roll_joint" type="continuous">
-    <parent link="link_pitch"/>
-    <child link="sphere_link"/>
+  <joint name="sphere_roll_joint" type="continuous">
+    <parent link="sphere_pitch"/>
+    <child link="sphere"/>
     <axis xyz="1 0 0"/>
     <origin xyz="0 0 0" rpy="0 0 0"/>
   </joint>
-  <gazebo reference="sphere_link">
+  <gazebo reference="sphere">
     <mu>10.0</mu>
     <mu2>10.0</mu2>
