Commit message: working movement

File: src/bb8_description/urdf/bb8.urdf.xacro (robot description, xacro)
@@ -4,3 +4,5 @@
   <xacro:include filename="hamster.xacro" />
   <xacro:include filename="sphere.xacro" />
+  <xacro:include filename="supports.xacro" />
+  <xacro:include filename="head.xacro" />
 </robot>

File: src/bb8_description/urdf/common_properties.xacro (robot description, xacro)
@@ -4,5 +4,5 @@
   <xacro:property name="base_radius" value="0.05" /> <!-- Radius of the circular base -->
   <xacro:property name="wheel_radius" value="0.069" /> <!-- Radius of the wheels -->
-  <xacro:property name="wheel_separation" value="0.364" /> <!-- Distance between the wheels -->
+  <xacro:property name="wheel_separation" value="0.3641" /> <!-- Distance between the wheels -->
   <xacro:property name="sphere_radius" value="0.51" /> <!-- Radius of the outer sphere -->
   <!-- Materials -->

File: src/bb8_description/urdf/hamster.xacro (robot description, xacro)
@@ -2,23 +2,37 @@
 <robot xmlns:xacro="http://www.ros.org/wiki/xacro">
   <link name="base_footprint" />
-  <!-- Circular Base Link -->
+  <!-- Base Link -->
   <link name="base_link">
     <visual>
+      <origin xyz="0 0 -${0.1458 + 0.025}" rpy="0 0 0"/>
       <geometry>
-        <mesh filename="file:///$(find bb8_description)/meshes/frame.stl" scale="0.001 0.001 0.001"/>
-        <!-- <cylinder length="0.01" radius="${base_radius}" /> -->
+        <!-- <mesh filename="file:///$(find bb8_description)/meshes/frame_b.stl" scale="0.000995 0.000995 0.000995"/> -->
+        <cylinder length="0.05" radius="0.09" />
       </geometry>
       <material name="blue"/>
     </visual>
-    <collision>
+    <!-- No need for collision -->
+    <!-- <collision>
       <geometry>
-        <!-- <mesh filename="file:///$(find bb8_description)/meshes/frame.stl" scale="0.001 0.001 0.0001"/> -->
-        <mesh filename="file:///$(find bb8_description)/meshes/frame.stl" scale="0.000999 0.000999 0.000999"/>
-        <!-- <cylinder length="0.01" radius="${base_radius}" /> -->
+        <mesh filename="file:///$(find bb8_description)/meshes/frame_b.stl" scale="0.000995 0.000995 0.000995"/>
       </geometry>
-    </collision>
+    </collision> -->
     <inertial>
-      <mass value="0.01"/>
+      <mass value="0.5"/>
       <inertia ixx="0.1" iyy="0.1" izz="0.1" ixy="0.0" ixz="0.0" iyz="0.0"/>
+    </inertial>
+  </link>
+  <link name="counterweight">
+    <visual>
+      <!-- STL origin is messed up, so need to move it -->
+      <origin xyz="0 0 ${0.19+0.05}" rpy="0 0 0"/>
+      <geometry>
+        <mesh filename="file:///$(find bb8_description)/meshes/counterweight.stl" scale="0.001 0.001 0.001"/>
+      </geometry>
+      <material name="black"/>
+    </visual>
+    <inertial>
+      <mass value="3.0"/>
+      <inertia ixx="1.0" iyy="1.0" izz="1.0" ixy="0.0" ixz="0.0" iyz="0.0"/>
     </inertial>
   </link>
@@ -26,16 +40,12 @@
   <link name="left_wheel">
     <visual>
-      <origin xyz="${wheel_separation/2 - 0.024} 0 0.1458" rpy="0 0 ${pi}"/>
       <geometry>
         <mesh filename="file:///$(find bb8_description)/meshes/wheel.stl" scale="0.001 0.001 0.001"/>
-        <!-- <cylinder length="0.025" radius="${wheel_radius}" /> -->
       </geometry>
       <material name="black"/>
     </visual>
     <collision>
-      <origin xyz="${wheel_separation/2 - 0.024} 0 0.1458" rpy="0 0 ${pi}"/>
       <geometry>
         <mesh filename="file:///$(find bb8_description)/meshes/wheel.stl" scale="0.001 0.001 0.001"/>
-        <!-- <cylinder length="0.025" radius="${wheel_radius}" /> -->
       </geometry>
     </collision>
@@ -48,16 +58,12 @@
   <link name="right_wheel">
     <visual>
-      <origin xyz="-${wheel_separation/2} 0 0.1458" rpy="0 0 0"/>
       <geometry>
         <mesh filename="file:///$(find bb8_description)/meshes/wheel.stl" scale="0.001 0.001 0.001"/>
-        <!-- <cylinder length="0.025" radius="${wheel_radius}" /> -->
       </geometry>
       <material name="black"/>
     </visual>
     <collision>
-      <origin xyz="-${wheel_separation/2} 0 0.1458" rpy="0 0 0"/>
       <geometry>
         <mesh filename="file:///$(find bb8_description)/meshes/wheel.stl" scale="0.001 0.001 0.001"/>
-        <!-- <cylinder length="0.025" radius="${wheel_radius}" /> -->
       </geometry>
     </collision>
@@ -73,15 +79,20 @@
       <origin xyz="0 0 0" rpy="0 0 0"/>
   </joint>
+  <joint name="counterweight_joint" type="fixed">
+      <parent link="base_link" />
+      <child link="counterweight" />
+      <origin xyz="0 0 -${0.19+0.05}" rpy="0 0 0"/>
+  </joint>
   <joint name="left_wheel_joint" type="continuous">
     <parent link="base_link"/>
     <child link="left_wheel"/>
-    <origin xyz="-${wheel_separation/2} 0 -0.1458" rpy="0 0 ${pi}"/>
-    <axis xyz="-1 0 0"/>
+    <origin xyz="${0.3437/2} 0 -0.1458" rpy="0 ${pi / 2} 0"/>
+    <axis xyz="0 0 1"/>
   </joint>
   <joint name="right_wheel_joint" type="continuous">
     <parent link="base_link"/>
     <child link="right_wheel"/>
-    <origin xyz="${wheel_separation/2} 0 -0.1458" rpy="0 0 0"/>
-    <axis xyz="1 0 0"/>
+    <origin xyz="-${0.3437/2} 0 -0.1458" rpy="0 ${pi/2} 0"/>
+    <axis xyz="0 0 1"/>
   </joint>
   <!-- Gazebo Plugins -->
@@ -103,16 +114,32 @@
   <!-- Collision Tuning for Robot and Sphere -->
   <gazebo reference="left_wheel">
-    <mu>100.0</mu>
-    <mu2>100.0</mu2>
-    <!-- <self_collide>true</self_collide> -->
+    <surface>
+      <contact>
+        <collide_without_contact>false</collide_without_contact>
+        <stiffness>1e6</stiffness>
+        <damping>2e3</damping>
+      </contact>
+      <friction>
+        <ode>
+          <mu>1.0</mu>
+          <mu2>1.0</mu2>
+        </ode>
+      </friction>
+    </surface>
   </gazebo>
   <gazebo reference="right_wheel">
-    <mu>100.0</mu>
-    <mu2>100.0</mu2>
-    <!-- <self_collide>true</self_collide> -->
-  </gazebo>
-  <gazebo reference="base_link">
-    <mu>0.01</mu>
-    <mu2>0.01</mu2>
+    <surface>
+      <contact>
+        <collide_without_contact>false</collide_without_contact>
+        <stiffness>1e6</stiffness>
+        <damping>2e3</damping>
+      </contact>
+      <friction>
+        <ode>
+          <mu>1.0</mu>
+          <mu2>1.0</mu2>
+        </ode>
+      </friction>
+    </surface>
   </gazebo>
 </robot>

File: src/bb8_description/urdf/sphere.xacro (robot description, xacro)
@@ -17,5 +17,5 @@
     </collision>
     <inertial>
-      <mass value="1"/>
+      <mass value="0.5"/>
       <inertia ixx="0.2" iyy="0.2" izz="0.2" ixy="0.0" ixz="0.0" iyz="0.0"/>
     </inertial>
@@ -26,5 +26,4 @@
     <child link="sphere_link"/>
     <origin xyz="0 0 0" rpy="0 0 0"/>
-    <!-- <origin xyz="0 0 ${sphere_radius}" rpy="0 0 0"/> -->
   </joint>
   <gazebo>
@@ -40,7 +39,10 @@
   </gazebo>
   <gazebo reference="sphere_link">
-    <mu>1.0</mu> <!-- Friction coefficient between sphere and ground -->
-    <mu2>1.0</mu2>
+    <mu>0.5</mu>
+    <mu2>0.5</mu2>
     <self_collide>true</self_collide>
+    <collision>
+      <margin>0.01</margin>
+    </collision>
   </gazebo>
 </robot>

Commit message: Now using ros2_control. Some problems with odom

File: src/bb8_description/urdf/bb8.urdf.xacro (robot description, xacro)
@@ -3,6 +3,9 @@
   <xacro:include filename="common_properties.xacro" />
   <xacro:include filename="hamster.xacro" />
-  <xacro:include filename="sphere.xacro" />
-  <xacro:include filename="supports.xacro" />
-  <xacro:include filename="head.xacro" />
+  <!-- <xacro:include filename="sphere.xacro" /> -->
+  <!-- <xacro:include filename="supports.xacro" /> -->
+  <!-- <xacro:include filename="head.xacro" /> -->
+  <xacro:include filename="gazebo_plugins.xacro" />
+  <xacro:include filename="ros2_control.xacro" />
+  <!-- <xacro:include filename="gazebo_control.xacro" /> -->
 </robot>

File: src/bb8_description/urdf/common_properties.xacro (robot description, xacro)
@@ -6,4 +6,23 @@
   <xacro:property name="wheel_separation" value="0.3641" /> <!-- Distance between the wheels -->
   <xacro:property name="sphere_radius" value="0.51" /> <!-- Radius of the outer sphere -->
+  <!-- Inertia -->
+  <xacro:macro name="inertial_sphere" params="mass radius *origin">
+      <inertial>
+          <xacro:insert_block name="origin"/>
+          <mass value="${mass}" />
+          <inertia ixx="${(2/5) * mass * (radius*radius)}" ixy="0.0" ixz="0.0"
+                  iyy="${(2/5) * mass * (radius*radius)}" iyz="0.0"
+                  izz="${(2/5) * mass * (radius*radius)}" />
+      </inertial>
+  </xacro:macro>
+  <xacro:macro name="inertial_cylinder" params="mass length radius *origin">
+    <inertial>
+        <xacro:insert_block name="origin"/>
+        <mass value="${mass}" />
+        <inertia ixx="${(1/12) * mass * (3*radius*radius + length*length)}" ixy="0.0" ixz="0.0"
+                iyy="${(1/12) * mass * (3*radius*radius + length*length)}" iyz="0.0"
+                izz="${(1/2) * mass * (radius*radius)}" />
+    </inertial>
+  </xacro:macro>
   <!-- Materials -->
   <material name="blue">

File: src/bb8_description/urdf/hamster.xacro (robot description, xacro)
@@ -1,4 +1,5 @@
 <?xml version="1.0"?>
 <robot xmlns:xacro="http://www.ros.org/wiki/xacro">
+  <!-- Base Footprint -->
   <link name="base_footprint" />
   <!-- Base Link -->
@@ -11,5 +12,9 @@
       <material name="blue"/>
     </visual>
+    <xacro:inertial_cylinder mass="0.5" length="0.05" radius="0.09">
+      <origin xyz="0 0 -${0.1458 + 0.025}" rpy="0 0 0"/>
+    </xacro:inertial_cylinder>
   </link>
+  <!-- Counterweight -->
   <link name="counterweight">
     <visual>
@@ -19,10 +24,9 @@
       <material name="black"/>
     </visual>
-    <inertial>
-      <mass value="3.0"/>
-      <inertia ixx="1.0" iyy="1.0" izz="1.0" ixy="0.0" ixz="0.0" iyz="0.0"/>
-    </inertial>
+    <xacro:inertial_cylinder mass="3.0" length="0.04" radius="0.05">
+      <origin xyz="0 0 0" rpy="0 0 0" />
+    </xacro:inertial_cylinder>
   </link>
-  <!-- Left Wheel Link -->
+  <!-- Left Wheel -->
   <link name="left_wheel">
     <visual>
@@ -37,10 +41,9 @@
       </geometry>
     </collision>
-    <inertial>
-      <mass value="0.05"/>
-      <inertia ixx="0.01" iyy="0.01" izz="0.01" ixy="0.0" ixz="0.0" iyz="0.0"/>
-    </inertial>
+    <xacro:inertial_sphere mass="0.05" radius="0.076">
+      <origin xyz="0 0 0" rpy="0 0 0"/>
+    </xacro:inertial_sphere>
   </link>
-  <!-- Right Wheel Link -->
+  <!-- Right Wheel -->
   <link name="right_wheel">
     <visual>
@@ -55,19 +58,18 @@
       </geometry>
     </collision>
-    <inertial>
-      <mass value="0.05"/>
-      <inertia ixx="0.01" iyy="0.01" izz="0.01" ixy="0.0" ixz="0.0" iyz="0.0"/>
-    </inertial>
+    <xacro:inertial_sphere mass="0.05" radius="0.076">
+      <origin xyz="0 0 0" rpy="0 0 0"/>
+    </xacro:inertial_sphere>
   </link>
   <!-- Joints -->
   <joint name="base_joint" type="fixed">
-      <parent link="base_footprint" />
-      <child link="base_link" />
-      <origin xyz="0 0 0" rpy="0 0 0"/>
+    <parent link="base_footprint" />
+    <child link="base_link" />
+    <origin xyz="0 0 0" rpy="0 0 0"/>
   </joint>
   <joint name="counterweight_joint" type="fixed">
-      <parent link="base_link" />
-      <child link="counterweight" />
-      <origin xyz="0 0 -0.21" rpy="0 0 0"/>
+    <parent link="base_link" />
+    <child link="counterweight" />
+    <origin xyz="0 0 -0.21" rpy="0 0 0"/>
   </joint>
   <joint name="left_wheel_joint" type="continuous">
@@ -83,20 +85,4 @@
     <axis xyz="0 0 1"/>
   </joint>
-  <!-- Gazebo Plugins -->
-  <gazebo>
-  <plugin name="diff_drive_controller" filename="libgazebo_ros_diff_drive.so">
-    <update_rate>50</update_rate>
-    <left_joint>left_wheel_joint</left_joint>
-    <right_joint>right_wheel_joint</right_joint>
-    <wheel_separation>${wheel_separation}</wheel_separation>
-    <wheel_diameter>${wheel_radius * 2}"</wheel_diameter>
-    <publish_odom>true</publish_odom>
-    <publish_odom_tf>true</publish_odom_tf>
-    <publish_wheel_tf>true</publish_wheel_tf>
-    <odometry_topic>odom</odometry_topic>
-    <odometry_frame>odom</odometry_frame>
-    <robot_base_frame>base_footprint</robot_base_frame>
-  </plugin>
-  </gazebo>
   <!-- Collision Tuning for Robot and Sphere -->
   <gazebo reference="left_wheel">

File: src/bb8_description/urdf/head.xacro (robot description, xacro)
@@ -17,8 +17,7 @@
       </geometry>
     </collision>
-    <inertial>
-      <mass value="1.0"/>
-      <inertia ixx="0.2" iyy="0.2" izz="0.2" ixy="0.0" ixz="0.0" iyz="0.0"/>
-    </inertial>
+    <xacro:inertial_cylinder mass="1.2" length="0.15" radius="0.15">
+        <origin xyz="0 0 0.045" rpy="0 0 0"/>
+    </xacro:inertial_cylinder>
   </link>
   <!-- Intermediate links for ball joint -->
@@ -58,10 +57,3 @@
     <origin xyz="0 0 0.26" rpy="0 0 0"/>
   </joint>
-  <gazebo>
-    <plugin name="gazebo_ros_joint_state_publisher" filename="libgazebo_ros_joint_state_publisher.so">
-      <joint_name>head_x_joint</joint_name>
-      <joint_name>head_y_joint</joint_name>
-      <update_rate>100.0</update_rate>
-    </plugin>
-  </gazebo>
 </robot>

File: src/bb8_description/urdf/sphere.xacro (robot description, xacro)
@@ -27,15 +27,4 @@
     <origin xyz="0 0 0" rpy="0 0 0"/>
   </joint>
-  <gazebo>
-  <plugin name="libgazebo_ros_p3d" filename="libgazebo_ros_p3d.so">
-    <ros>
-      <remapping>odom:=sphere_pose</remapping>
-    </ros>
-    <frame_name>base_footprint</frame_name>
-    <body_name>sphere_link</body_name>
-    <update_rate>50</update_rate>
-    <gaussian_noise>0.01</gaussian_noise>
-    </plugin>
-  </gazebo>
   <gazebo reference="sphere_link">
     <mu>0.5</mu>

File: src/bb8_description/urdf/supports.xacro (robot description, xacro)
@@ -4,5 +4,5 @@
   <link name="supports"/>
   <!-- Macro to create individual supports -->
-  <xacro:macro name="spherical_support" params="prefix angle">
+  <xacro:macro name="spherical_support" params="prefix angle_1 angle_2">
     <!-- Virtual link for positioning -->
     <link name="${prefix}_virtual"/>
@@ -29,5 +29,5 @@
       <parent link="supports"/>
       <child link="${prefix}_virtual"/>
-      <origin xyz="0 0 0" rpy="0 ${pi / 4} ${angle}"/>
+      <origin xyz="0 0 0" rpy="0 ${angle_1} ${angle_2}"/>
     </joint>
     <joint name="${prefix}_sphere_joint" type="fixed">
@@ -48,8 +48,6 @@
     </gazebo>
   </xacro:macro>
-  <!-- <xacro:spherical_support prefix="support1" angle="$(eval 0)"/> -->
-  <xacro:spherical_support prefix="support2" angle="$(eval 2*pi/4)"/>
-  <!-- <xacro:spherical_support prefix="support3" angle="$(eval 4*pi/4)"/> -->
-  <xacro:spherical_support prefix="support4" angle="$(eval 6*pi/4)"/>
+  <xacro:spherical_support prefix="support1" angle_1="$(eval pi/4)" angle_2="$(eval 2*pi/4)"/>
+  <xacro:spherical_support prefix="support2" angle_1="$(eval pi/4)" angle_2="$(eval 6*pi/4)"/>
   <!-- Connect supports to base -->
   <joint name="supports_joint" type="fixed">

Commit message: Added controller to head joints

File: src/bb8_description/urdf/bb8.urdf.xacro (robot description, xacro)
@@ -3,7 +3,7 @@
   <xacro:include filename="common_properties.xacro" />
   <xacro:include filename="hamster.xacro" />
-  <!-- <xacro:include filename="sphere.xacro" /> -->
-  <!-- <xacro:include filename="supports.xacro" /> -->
-  <!-- <xacro:include filename="head.xacro" /> -->
+  <xacro:include filename="sphere.xacro" />
+  <xacro:include filename="supports.xacro" />
+  <xacro:include filename="head.xacro" />
   <xacro:include filename="gazebo_plugins.xacro" />
   <xacro:include filename="ros2_control.xacro" />

File: src/bb8_description/urdf/gazebo_plugins.xacro (robot description, xacro)
@@ -1,13 +1,13 @@
 <?xml version="1.0"?>
 <robot xmlns:xacro="http://www.ros.org/wiki/xacro">
-  <gazebo>
+  <!-- <gazebo>
     <plugin name="gazebo_ros_joint_state_publisher" filename="libgazebo_ros_joint_state_publisher.so">
-      <!-- <joint_name>right_wheel_joint</joint_name> -->
-      <!-- <joint_name>left_wheel_joint</joint_name> -->
+      <joint_name>right_wheel_joint</joint_name>
+      <joint_name>left_wheel_joint</joint_name>
       <joint_name>head_x_joint</joint_name>
       <joint_name>head_y_joint</joint_name>
       <update_rate>100.0</update_rate>
     </plugin>
-  </gazebo>
+  </gazebo> -->
   <gazebo>
     <plugin name="libgazebo_ros_p3d" filename="libgazebo_ros_p3d.so">

File: src/bb8_description/urdf/ros2_control.xacro (robot description, xacro)
@@ -21,4 +21,18 @@
             <state_interface name="position"/>
         </joint>
+        <joint name="head_x_joint">
+            <command_interface name="position">
+                <param name="min">-20</param>
+                <param name="max">20</param>
+            </command_interface>
+            <state_interface name="position"/>
+        </joint>
+        <joint name="head_y_joint">
+            <command_interface name="position">
+                <param name="min">-20</param>
+                <param name="max">20</param>
+            </command_interface>
+            <state_interface name="position"/>
+        </joint>
     </ros2_control>
     <gazebo>

File: src/bb8_description/urdf/supports.xacro (robot description, xacro)
@@ -50,4 +50,7 @@
   <xacro:spherical_support prefix="support1" angle_1="$(eval pi/4)" angle_2="$(eval 2*pi/4)"/>
   <xacro:spherical_support prefix="support2" angle_1="$(eval pi/4)" angle_2="$(eval 6*pi/4)"/>
+  <xacro:spherical_support prefix="support3" angle_1="$(eval -pi/3)" angle_2="$(eval 0)"/>
+  <xacro:spherical_support prefix="support4" angle_1="$(eval -pi/3)" angle_2="$(eval 2*pi/3)"/>
+  <xacro:spherical_support prefix="support5" angle_1="$(eval -pi/3)" angle_2="$(eval 4*pi/3)"/>
   <!-- Connect supports to base -->
   <joint name="supports_joint" type="fixed">
