Commit message: Added lidar and tried slam

File: src/bb8_description/urdf/bb8.urdf.xacro (robot description, xacro)
@@ -9,4 +9,5 @@
   <xacro:include filename="ros2_control.xacro" />
   <xacro:include filename="sensors.xacro" />
+  <xacro:include filename="lidar.xacro" />
   <!-- <xacro:include filename="gazebo_control.xacro" /> -->
 </robot>

File: src/bb8_description/urdf/hamster.xacro (robot description, xacro)
@@ -24,5 +24,5 @@
       <material name="black"/>
     </visual>
-    <xacro:inertial_cylinder mass="3.0" length="0.04" radius="0.05">
+    <xacro:inertial_cylinder mass="1.0" length="0.04" radius="0.05">
       <origin xyz="0 0 0" rpy="0 0 0" />
     </xacro:inertial_cylinder>
@@ -31,4 +31,5 @@
   <link name="left_wheel">
     <visual>
+      <origin xyz="0 0 0" rpy="0 ${pi/2} 0"/>
       <geometry>
         <mesh filename="file:///$(find bb8_description)/meshes/wheel.stl" scale="0.001 0.001 0.001"/>
@@ -37,4 +38,5 @@
     </visual>
     <collision>
+      <origin xyz="0 0 0" rpy="0 ${pi/2} 0"/>
       <geometry>
         <mesh filename="file:///$(find bb8_description)/meshes/wheel.stl" scale="0.001 0.001 0.001"/>
@@ -42,10 +44,22 @@
     </collision>
     <xacro:inertial_sphere mass="0.05" radius="0.076">
+      <origin xyz="0 0 0" rpy="0 ${pi/2} 0"/>
+    </xacro:inertial_sphere>
+  </link>
+  <link name="wheel_connector" >
+    <visual>
+      <geometry>
+        <cylinder length="0.01" radius="0.01" />
+      </geometry>
+      <material name="blue"/>
+    </visual>
+    <xacro:inertial_cylinder mass="0.01" length="0.01" radius="0.01">
       <origin xyz="0 0 0" rpy="0 0 0"/>
-    </xacro:inertial_sphere>
+    </xacro:inertial_cylinder>
   </link>
   <!-- Right Wheel -->
   <link name="right_wheel">
     <visual>
+      <origin xyz="0 0 0" rpy="0 ${pi/2} 0"/>
       <geometry>
         <mesh filename="file:///$(find bb8_description)/meshes/wheel.stl" scale="0.001 0.001 0.001"/>
@@ -54,4 +68,5 @@
     </visual>
     <collision>
+      <origin xyz="0 0 0" rpy="0 ${pi/2} 0"/>
       <geometry>
         <mesh filename="file:///$(find bb8_description)/meshes/wheel.stl" scale="0.001 0.001 0.001"/>
@@ -59,5 +74,5 @@
     </collision>
     <xacro:inertial_sphere mass="0.05" radius="0.076">
-      <origin xyz="0 0 0" rpy="0 0 0"/>
+      <origin xyz="0 0 0" rpy="0 ${pi/2} 0"/>
     </xacro:inertial_sphere>
   </link>
@@ -68,4 +83,9 @@
     <origin xyz="0 0 0" rpy="0 0 0"/>
   </joint>
+  <joint name="wheel_connector_joint" type="fixed">
+    <parent link="base_link" />
+    <child link="wheel_connector" />
+    <origin xyz="0 0 0" rpy="0 0 ${pi/2}"/>
+  </joint>
   <joint name="counterweight_joint" type="fixed">
     <parent link="base_link" />
@@ -74,14 +94,14 @@
   </joint>
   <joint name="left_wheel_joint" type="continuous">
-    <parent link="base_link"/>
+    <parent link="wheel_connector"/>
     <child link="left_wheel"/>
-    <origin xyz="${0.3437/2} 0 -0.1458" rpy="0 ${pi / 2} 0"/>
-    <axis xyz="0 0 1"/>
+    <origin xyz="${0.3437/2} 0 -0.1458" rpy="0 0 0"/>
+    <axis xyz="1 0 0"/>
   </joint>
   <joint name="right_wheel_joint" type="continuous">
-    <parent link="base_link"/>
+    <parent link="wheel_connector"/>
     <child link="right_wheel"/>
-    <origin xyz="-${0.3437/2} 0 -0.1458" rpy="0 ${pi/2} 0"/>
-    <axis xyz="0 0 1"/>
+    <origin xyz="-${0.3437/2} 0 -0.1458" rpy="0 0 0"/>
+    <axis xyz="1 0 0"/>
   </joint>
   <!-- Collision Tuning for Robot and Sphere -->

File: src/bb8_description/urdf/head.xacro (robot description, xacro)
@@ -11,11 +11,11 @@
       </material>
     </visual>
-    <collision>
+    <!-- <collision>
       <origin xyz="0 0 -0.26" rpy="0 0 0"/>
       <geometry>
         <mesh filename="file:///$(find bb8_description)/meshes/head.stl" scale="0.001 0.001 0.001"/>
       </geometry>
-    </collision>
-    <xacro:inertial_cylinder mass="1.2" length="0.15" radius="0.15">
+    </collision> -->
+    <xacro:inertial_cylinder mass="0.5" length="0.15" radius="0.15">
         <origin xyz="0 0 0.045" rpy="0 0 0"/>
     </xacro:inertial_cylinder>

File: src/bb8_description/urdf/sensors.xacro (robot description, xacro)
@@ -42,5 +42,5 @@
     </gazebo>
   </xacro:macro>
-    <xacro:imu_sensor parent_link="base_link" sensor_name="imu_base"/>
-    <xacro:imu_sensor parent_link="head" sensor_name="imu_head"/>
+  <xacro:imu_sensor parent_link="base_link" sensor_name="imu_base"/>
+  <xacro:imu_sensor parent_link="head" sensor_name="imu_head"/>
 </robot>

File: src/bb8_description/urdf/sphere.xacro (robot description, xacro)
@@ -27,5 +27,5 @@
     <origin xyz="0 0 0" rpy="0 0 0"/>
   </joint>
-  <gazebo reference="sphere_link">
+  <!-- <gazebo reference="sphere_link">
     <mu>0.5</mu>
     <mu2>0.5</mu2>
@@ -33,4 +33,18 @@
       <margin>0.01</margin>
     </collision>
-  </gazebo>
+  </gazebo> -->
+  <gazebo reference="sphere_link">
+    <mu>1.0</mu>
+    <mu2>1.0</mu2>
+    <collision>
+      <surface>
+        <contact>
+          <ode>
+            <min_depth>0.001</min_depth>
+            </ode>
+        </contact>
+      </surface>
+      <margin>0.01</margin>
+    </collision>
+   </gazebo>
 </robot>

File: src/bb8_description/urdf/supports.xacro (robot description, xacro)
@@ -34,20 +34,24 @@
       <parent link="${prefix}_virtual"/>
       <child link="${prefix}_sphere"/>
-      <origin xyz="0.249 0 0" rpy="0 0 0"/>
+      <origin xyz="0.2494 0 0" rpy="0 0 0"/>
     </joint>
     <!-- Physics properties -->
     <gazebo reference="${prefix}_sphere">
-      <mu>0.01</mu>
-      <mu2>0.01</mu2>
+      <mu>0.001</mu>
+      <mu2>0.001</mu2>
       <self_collide>true</self_collide>
       <contact>
         <collide_without_contact>false</collide_without_contact>
-        <stiffness>5e6</stiffness>
-        <damping>1e3</damping>
+        <stiffness>1e3</stiffness>
+        <damping>10</damping>
       </contact>
     </gazebo>
   </xacro:macro>
-  <xacro:spherical_support prefix="support1" angle_1="$(eval pi/4)" angle_2="$(eval 2*pi/4)"/>
-  <xacro:spherical_support prefix="support2" angle_1="$(eval pi/4)" angle_2="$(eval 6*pi/4)"/>
+  <xacro:spherical_support prefix="support1" angle_1="$(eval pi/4)" angle_2="$(eval 0)"/>
+  <xacro:spherical_support prefix="support2" angle_1="$(eval pi/4)" angle_2="$(eval 4*pi/4)"/>
+  <!-- <xacro:spherical_support prefix="support1" angle_1="$(eval pi/4)" angle_2="$(eval pi/4)"/> -->
+  <!-- <xacro:spherical_support prefix="support2" angle_1="$(eval pi/4)" angle_2="$(eval 3*pi/4)"/> -->
+  <!-- <xacro:spherical_support prefix="support6" angle_1="$(eval pi/4)" angle_2="$(eval 5*pi/4)"/> -->
+  <!-- <xacro:spherical_support prefix="support7" angle_1="$(eval pi/4)" angle_2="$(eval 7*pi/4)"/> -->
   <xacro:spherical_support prefix="support3" angle_1="$(eval -pi/3)" angle_2="$(eval 0)"/>
   <xacro:spherical_support prefix="support4" angle_1="$(eval -pi/3)" angle_2="$(eval 2*pi/3)"/>

Commit message: tuned sim params, better map

File: src/bb8_description/urdf/bb8.urdf.xacro (robot description, xacro)
@@ -9,4 +9,3 @@
   <xacro:include filename="sensors.xacro" />
   <xacro:include filename="lidar.xacro" />
-  <!-- <xacro:include filename="gazebo_control.xacro" /> -->
 </robot>

File: src/bb8_description/urdf/hamster.xacro (robot description, xacro)
@@ -114,6 +114,6 @@
       <contact>
         <ode>
-          <min_depth>0.05</min_depth>
-          <margin>0.05</margin>
+          <min_depth>0.001</min_depth>
+          <margin>0.001</margin>
         </ode>
         <collide_without_contact>false</collide_without_contact>
@@ -134,6 +134,6 @@
       <contact>
         <ode>
-          <min_depth>0.05</min_depth>
-          <margin>0.05</margin>
+          <min_depth>0.001</min_depth>
+          <margin>0.001</margin>
         </ode>
         <collide_without_contact>false</collide_without_contact>

File: src/bb8_description/urdf/sphere.xacro (robot description, xacro)
@@ -34,9 +34,9 @@
       <contact>
         <ode>
-          <min_depth>0.01</min_depth>
-          <margin>0.02</margin>
+          <min_depth>0.001</min_depth>
+          <margin>0.001</margin>
         </ode>
-        <stiffness>1e3</stiffness>     <!-- Contact stiffness -->
-        <damping>1e2</damping>         <!-- Contact damping -->
+        <stiffness>1e5</stiffness>     <!-- Contact stiffness -->
+        <damping>1e3</damping>         <!-- Contact damping -->
       </contact>
     </surface>

File: src/bb8_description/urdf/supports.xacro (robot description, xacro)
@@ -34,5 +34,5 @@
       <parent link="${prefix}_virtual"/>
       <child link="${prefix}_sphere"/>
-      <origin xyz="0.2494 0 0" rpy="0 0 0"/>
+      <origin xyz="0.249 0 0" rpy="0 0 0"/>
     </joint>
     <!-- Physics properties -->
@@ -45,5 +45,5 @@
           <ode>
             <min_depth>0.01</min_depth>  <!-- Minimum penetration depth for collision response -->
-            <margin>0.02</margin>        <!-- Distance buffer for collision detection -->
+            <margin>0.01</margin>        <!-- Distance buffer for collision detection -->
           </ode>
           <stiffness>1e6</stiffness>     <!-- Contact stiffness -->
@@ -51,19 +51,20 @@
         </contact>
       </surface>
+      <collide_without_contact>false</collide_without_contact>
     </gazebo>
   </xacro:macro>
-  <!-- <xacro:spherical_support prefix="support1" angle_1="$(eval pi/4)" angle_2="$(eval 0)"/> -->
-  <!-- <xacro:spherical_support prefix="support2" angle_1="$(eval pi/4)" angle_2="$(eval 4*pi/4)"/> -->
-  <xacro:spherical_support prefix="support3" angle_1="$(eval pi/4)" angle_2="$(eval pi/4)"/>
+  <!-- <xacro:spherical_support prefix="support1" angle_1="$(eval pi/4)" angle_2="$(eval 0)"/>
+  <xacro:spherical_support prefix="support2" angle_1="$(eval pi/4)" angle_2="$(eval 4*pi/4)"/> -->
+  <!-- <xacro:spherical_support prefix="support3" angle_1="$(eval pi/4)" angle_2="$(eval pi/4)"/>
   <xacro:spherical_support prefix="support4" angle_1="$(eval pi/4)" angle_2="$(eval 3*pi/4)"/>
   <xacro:spherical_support prefix="support5" angle_1="$(eval pi/4)" angle_2="$(eval 5*pi/4)"/>
-  <xacro:spherical_support prefix="support6" angle_1="$(eval pi/4)" angle_2="$(eval 7*pi/4)"/>
+  <xacro:spherical_support prefix="support6" angle_1="$(eval pi/4)" angle_2="$(eval 7*pi/4)"/> -->
   <xacro:spherical_support prefix="support7" angle_1="$(eval -pi/3)" angle_2="$(eval 0)"/>
   <xacro:spherical_support prefix="support8" angle_1="$(eval -pi/3)" angle_2="$(eval 2*pi/3)"/>
   <xacro:spherical_support prefix="support9" angle_1="$(eval -pi/3)" angle_2="$(eval 4*pi/3)"/>
-  <!-- <xacro:spherical_support prefix="support10" angle_1="$(eval -pi/3)" angle_2="$(eval 0)"/> -->
-  <!-- <xacro:spherical_support prefix="support11" angle_1="$(eval -pi/3)" angle_2="$(eval pi/2)"/> -->
-  <!-- <xacro:spherical_support prefix="support12" angle_1="$(eval -pi/3)" angle_2="$(eval pi)"/> -->
-  <!-- <xacro:spherical_support prefix="support13" angle_1="$(eval -pi/3)" angle_2="$(eval 3*pi/2)"/> -->
+  <xacro:spherical_support prefix="support10" angle_1="$(eval -pi/3)" angle_2="$(eval 0)"/>
+  <xacro:spherical_support prefix="support11" angle_1="$(eval -pi/3)" angle_2="$(eval pi/2)"/>
+  <xacro:spherical_support prefix="support12" angle_1="$(eval -pi/3)" angle_2="$(eval pi)"/>
+  <xacro:spherical_support prefix="support13" angle_1="$(eval -pi/3)" angle_2="$(eval 3*pi/2)"/>
   <!-- Connect supports to base -->
   <joint name="supports_joint" type="fixed">

Commit message: Fixed turning!

File: src/bb8_description/urdf/bb8.urdf.xacro (robot description, xacro)
@@ -4,5 +4,4 @@
   <xacro:include filename="hamster.xacro" />
   <xacro:include filename="sphere.xacro" />
-  <xacro:include filename="supports.xacro" />
   <xacro:include filename="head.xacro" />
   <xacro:include filename="ros2_control.xacro" />

File: src/bb8_description/urdf/hamster.xacro (robot description, xacro)
@@ -5,6 +5,4 @@
   <link name="base_footprint" />
   <link name="sphere_center" />
-  <!-- <link name="base_roll" /> -->
-  <!-- <link name="base_pitch" /> -->
   <!-- Base Link -->
   <link name="base_link">

File: src/bb8_description/urdf/sphere.xacro (robot description, xacro)
@@ -1,4 +1,17 @@
 <?xml version="1.0"?>
 <robot xmlns:xacro="http://www.ros.org/wiki/xacro">
+  <!-- Dummy links for rotational joints -->
+  <link name="link_yaw">
+    <inertial>
+      <mass value="0.001"/>
+      <inertia ixx="0.0001" iyy="0.0001" izz="0.0001" ixy="0" ixz="0" iyz="0"/>
+    </inertial>
+  </link>
+  <link name="link_pitch">
+    <inertial>
+      <mass value="0.001"/>
+      <inertia ixx="0.0001" iyy="0.0001" izz="0.0001" ixy="0" ixz="0" iyz="0"/>
+    </inertial>
+  </link>
   <!-- Outer Sphere Link -->
   <link name="sphere_link">
@@ -21,8 +34,22 @@
     </inertial>
   </link>
-  <!-- Joint to Connect Sphere and Hamster -->
-  <joint name="sphere_joint" type="floating">
+  <!-- Continuous joints -->
+  <joint name="yaw_joint" type="continuous">
     <parent link="sphere_center"/>
+    <child link="link_yaw"/>
+    <axis xyz="0 0 1"/>
+    <origin xyz="0 0 0" rpy="0 0 0"/>
+  </joint>
+  <joint name="pitch_joint" type="continuous">
+    <parent link="link_yaw"/>
+    <child link="link_pitch"/>
+    <axis xyz="0 1 0"/>
+    <origin xyz="0 0 0" rpy="0 0 0"/>
+  </joint>
+  <joint name="roll_joint" type="continuous">
+    <parent link="link_pitch"/>
     <child link="sphere_link"/>
+    <axis xyz="1 0 0"/>
+    <origin xyz="0 0 0" rpy="0 0 0"/>
   </joint>
   <gazebo reference="sphere_link">

Commit message: added camera and z revolute joint for head

File: src/bb8_description/urdf/bb8.urdf.xacro (robot description, xacro)
@@ -8,3 +8,4 @@
   <xacro:include filename="sensors.xacro" />
   <xacro:include filename="lidar.xacro" />
+  <xacro:include filename="camera.xacro" />
 </robot>

File: src/bb8_description/urdf/head.xacro (robot description, xacro)
@@ -51,9 +51,11 @@
     <dynamics damping="0.1" friction="0.01"/>
   </joint>
-  <!-- Fixed joint to attach head to the final rotation link -->
-  <joint name="head_attachment" type="fixed">
+  <!-- Continuous revolute joint for z -->
+  <joint name="head_z_joint" type="continuous">
     <parent link="head_y_link"/>
     <child link="head"/>
     <origin xyz="0 0 0.26" rpy="0 0 0"/>
+    <axis xyz="0 0 1"/>
+    <dynamics damping="0.1" friction="0.01"/>
   </joint>
 </robot>

File: src/bb8_description/urdf/ros2_control.xacro (robot description, xacro)
@@ -35,4 +35,12 @@
             <state_interface name="position"/>
         </joint>
+        <joint name="head_z_joint">
+            <command_interface name="velocity">
+                <param name="min">-5.0</param>
+                <param name="max">5.0</param>
+            </command_interface>
+            <state_interface name="velocity"/>
+            <state_interface name="position"/>
+        </joint>
     </ros2_control>
     <gazebo>
