Commit message: fixed camera orientation

File: src/bb8_description/urdf/camera.xacro (robot description, xacro)
@@ -1,55 +1,47 @@
 <?xml version="1.0"?>
 <robot xmlns:xacro="http://www.ros.org/wiki/xacro">
-  <!-- Fixed joint to attach the camera to the front of the head -->
-  <joint name="camera_joint" type="fixed">
-    <parent link="head"/>
-    <child link="camera"/>
-    <origin xyz="0.15 0 0.075" rpy="0 0 0"/>
-  </joint>
-  <!-- Camera Link Definition -->
-  <link name="camera">
-    <!-- Visual Representation -->
-    <visual>
-      <geometry>
-        <!-- Simple box to represent a camera -->
-        <box size="0.04 0.04 0.02"/>
-      </geometry>
-      <material name="black"/>
-    </visual>
-    <!-- Inertial Properties (lightweight sensor) -->
-    <inertial>
-      <mass value="0.05"/> <!-- Lighter than lidar -->
-      <origin xyz="0 0 0"/>
-      <inertia ixx="0.0001" iyy="0.0001" izz="0.0001" ixy="0" ixz="0" iyz="0"/>
-    </inertial>
-  </link>
-  <!-- Gazebo Sensor Plugin -->
-  <gazebo reference="camera">
-    <sensor name="camera_sensor" type="camera">
-      <visualize>true</visualize>
-      <update_rate>30.0</update_rate> <!-- Higher rate for smoother video -->
-      <!-- Camera Properties -->
-      <camera>
-        <horizontal_fov>${pi/2}</horizontal_fov> <!-- 90 degrees FOV -->
-        <image>
-          <width>640</width>
-          <height>480</height>
-          <format>R8G8B8</format>
-        </image>
-        <clip>
-          <near>0.02</near>
-          <far>10.0</far>
-        </clip>
-      </camera>
-      <!-- ROS Integration -->
-      <plugin name="camera_plugin" filename="libgazebo_ros_camera_sensor.so">
-        <ros>
-          <remapping>~/image:=image_raw</remapping>
-        </ros>
-        <frame_name>camera</frame_name>
-        <topic_name>camera/image_raw</topic_name>
-        <hack_baseline>0.07</hack_baseline> <!-- Optional for stereo -->
-      </plugin>
-    </sensor>
-  </gazebo>
+    <xacro:property name="camera_length" value="0.01" />
+    <xacro:property name="camera_width" value="0.1" />
+    <xacro:property name="camera_height" value="0.05" />
+    <link name="camera_link">
+        <visual>
+            <geometry>
+                <box size="${camera_length} ${camera_width} ${camera_height}" />
+            </geometry>
+            <material name="grey" />
+        </visual>
+        <collision>
+            <geometry>
+                <box size="${camera_length} ${camera_width} ${camera_height}" />
+            </geometry>
+        </collision>
+        <xacro:inertial_box m="0.1" l="${camera_length}" w="${camera_width}" h="${camera_height}"
+                           xyz="0 0 0" rpy="0 0 0" />
+    </link>
+    <joint name="base_camera_joint" type="fixed">
+        <parent link="head" />
+        <child link="camera_link" />
+        <origin xyz="0.15 0 0.075" rpy="0 0 0" />
+    </joint>
+    <link name="camera_link_optical">
+    </link>
+    <joint name="camera_optical_joint" type="fixed">
+        <!-- these values have to be these values otherwise the gazebo camera
+            image won't be aligned properly with the frame it is supposedly
+            originating from -->
+        <origin xyz="0 0 0" rpy="${-pi/2} 0 ${-pi/2}"/>
+        <parent link="camera_link"/>
+        <child link="camera_link_optical"/>
+    </joint>
+    <gazebo reference="camera_link">
+        <material>Gazebo/Red</material>
+        <sensor name="camera_sensor" type="camera">
+            <pose>0 0 0 0 0 0</pose>
+            <visualize>false</visualize>
+            <update_rate>10.0</update_rate>
+            <plugin name="camera_controller" filename="libgazebo_ros_camera.so">
+                <frame_name>camera_link_optical</frame_name>
+            </plugin>
+        </sensor>
+    </gazebo>
 </robot>

File: src/bb8_description/urdf/common_properties.xacro (robot description, xacro)
@@ -26,4 +26,13 @@
     </inertial>
   </xacro:macro>
+  <xacro:macro name="inertial_box" params="m l w h xyz rpy">
+      <inertial>
+          <origin xyz="${xyz}" rpy="${rpy}" />
+          <mass value="${m}" />
+          <inertia ixx="${(m/12) * (h*h + l*l)}" ixy="0" ixz="0"
+                    iyy="${(m/12) * (w*w + l*l)}" iyz="0"
+                    izz="${(m/12) * (w*w + h*h)}" />
+      </inertial>
+  </xacro:macro>
   <!-- Materials -->
   <material name="blue">

Commit message: Red_circle_follower complete

File: src/bb8_description/urdf/camera.xacro (robot description, xacro)
@@ -1,7 +1,9 @@
 <?xml version="1.0"?>
 <robot xmlns:xacro="http://www.ros.org/wiki/xacro">
+    <!-- Camera Dimensions -->
     <xacro:property name="camera_length" value="0.01" />
     <xacro:property name="camera_width" value="0.1" />
     <xacro:property name="camera_height" value="0.05" />
+    <!-- Camera Link -->
     <link name="camera_link">
         <visual>
@@ -19,4 +21,5 @@
                            xyz="0 0 0" rpy="0 0 0" />
     </link>
+    <!-- Fixed Joint from Head to Camera Link -->
     <joint name="base_camera_joint" type="fixed">
         <parent link="head" />
@@ -24,14 +27,12 @@
         <origin xyz="0.15 0 0.075" rpy="0 0 0" />
     </joint>
-    <link name="camera_link_optical">
-    </link>
+    <!-- Optical Frame (for ROS camera conventions) -->
+    <link name="camera_link_optical" />
     <joint name="camera_optical_joint" type="fixed">
-        <!-- these values have to be these values otherwise the gazebo camera
-            image won't be aligned properly with the frame it is supposedly
-            originating from -->
-        <origin xyz="0 0 0" rpy="${-pi/2} 0 ${-pi/2}"/>
         <parent link="camera_link"/>
         <child link="camera_link_optical"/>
+        <origin xyz="0 0 0" rpy="${-pi/2} 0 ${-pi/2}"/>
     </joint>
+    <!-- Gazebo Camera Sensor -->
     <gazebo reference="camera_link">
         <material>Gazebo/Red</material>
@@ -40,4 +41,18 @@
             <visualize>false</visualize>
             <update_rate>10.0</update_rate>
+            <!-- Camera Parameters -->
+            <camera>
+                <horizontal_fov>1.0472</horizontal_fov> <!-- 60 degrees in radians -->
+                <image>
+                    <width>640</width>
+                    <height>480</height>
+                    <format>R8G8B8</format>
+                </image>
+                <clip>
+                    <near>0.02</near>
+                    <far>10.0</far>
+                </clip>
+            </camera>
+            <!-- ROS Integration -->
             <plugin name="camera_controller" filename="libgazebo_ros_camera.so">
                 <frame_name>camera_link_optical</frame_name>
